File: AquaMaster-Carrier.brd (EAGLE design)
At the start: 46 x 35.3 mm, 44 parts, among them J2 5V @ 2A, Q1 BSS138, Q2 BSS138, Q3 BSS138, Q4 BSS138

Commit message: Latest AquaMaster Carrier Board - sent to OSHPark today
Parts:
- removed JP2: VSelect, SparkFun-Jumpers:SMT-JUMPER_3_1-NC_PASTE_SILK
- removed Q1, Q2, Q3, Q4: BSS138, SparkFun:SOT23-3
- removed R1, R10, R11, R12, R4, R6, R8, R9: 10K, adafruit:R0805
- removed SPI: (no value), SparkFun-Connectors:1X06_LOCK
- added FLOW: (no value), SparkFun-Connectors:1X03_LOCK
- moved R2 13.3 mm to (20.6, 18.7), turned to 90 degrees
- moved V1 13.3 mm to (31.9, 32.0), turned to 90 degrees
- moved R7 12.5 mm to (16.3, 15.2)
- moved R5 12.5 mm to (25.4, 20.2)
- moved WATCHDOG 12.4 mm to (16.5, 18.4)
- moved R3 12.4 mm to (25.4, 23.0)
- moved JP1 12.0 mm to (22.9, 13.7)
- moved F1 8.70 mm to (35.1, 31.5), turned to 90 degrees
- moved V2 8.02 mm to (17.4, 3.17)
- moved 12V-5V-BUCK 5.09 mm to (31.6, 3.94), turned to 0 degrees
- moved J1 3.58 mm to (25.1, 3.94), turned to 0 degrees
- moved F2 3.56 mm to (19.8, 4.19)
Connections:
- removed net A2-EXT: Q1.3, R4.2, SPI.2
- removed net A3: PHOTON.9, Q2.2, R6.2
- removed net A3-EXT: Q2.3, R8.2, SPI.3
- removed net A4: PHOTON.8, Q3.2, R9.2
- removed net A4-EXT: Q3.3, R10.2, SPI.4
- removed net A5: PHOTON.7, Q4.2, R11.2
- removed net A5-EXT: Q4.3, R12.2, SPI.5
- removed net VIO-EXT: F2.2, SPI.6, V2.2
- removed net VSELECT: F2.1, JP2.2, R10.1, R12.1, R4.1, R8.1
- new net LED: PHOTON.20
- new net VIN-EXT: F2.2, FLOW.3, V2.2
- net A2: now also FLOW.2; no longer Q1.2, R1.2
- net DONE: now also PHOTON.15; no longer PHOTON.19
- net GND: now also FLOW.1; no longer SPI.1
- net SOLENOID: now also PHOTON.19; no longer PHOTON.15
- net VCC: no longer JP2.3, Q1.1, Q2.1, Q3.1, Q4.1, R1.1, R11.1, R13.2, R14.2, R6.1, R9.1
- net VCC-EXT: now also R13.2, R14.2
- net VIN: now also F2.1; no longer JP2.1
Routing:
- net VCC: track 89.1 -> 28.5 mm
- net VSELECT: track 34.0 -> 0.00 mm, vias 2 -> 0
- net A2-EXT: track 20.8 -> 0.00 mm, vias 2 -> 0
- net A5-EXT: track 20.2 -> 0.00 mm, vias 2 -> 0
- net A3-EXT: track 19.5 -> 0.00 mm, vias 2 -> 0
- net A4-EXT: track 19.4 -> 0.00 mm, vias 2 -> 0
- net !RST: track 11.9 -> 26.4 mm
- net GATE: track 19.1 -> 6.80 mm
- net A5: track 8.03 -> 0.00 mm
- net A3: track 7.57 -> 0.00 mm
- net VIN: track 16.3 -> 23.9 mm, vias 0 -> 1
- net A4: track 7.40 -> 0.00 mm
- net WAKE: track 16.2 -> 22.0 mm, vias 1 -> 0
- net VIN-EXT: track 0.00 -> 5.36 mm
- net VIO-EXT: track 4.97 -> 0.00 mm
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Other:
- board text added: "DC-IN - 12V @3A Vin - 5V @1.5A Vcc - 3.3v @ 100mA"
- board text added: "DC-IN GND VIN"
- board text added: "VCC SCL SDA GND"
- board text added: "VIN A2 GND"
- board text added: "chip@seeinsights.com 8-22-17 AquaMaster Carrier v2"
- board text removed: "OUT GND IN"
- board text removed: "VCC A5 A4 A3 A2 GND"
- board text removed: "chip@seeinsights.com 8-22-17 Photon Carrier v2"

Commit message: Added BOM
Parts:
- removed JP1: DOG-SW, SparkFun-Jumpers:SMT-JUMPER_2_NO_NO-SILK
- added LOGO1: OSHW-LOGOS, SparkFun-Aesthetics:OSHW-LOGO-S
- added R1: 97.6k, adafruit:R0805
- R2: value 25k -> 100k
- moved J1 1.91 mm to (23.2, 3.94)
- moved R2 1.40 mm to (19.2, 18.7)
- moved WATCHDOG 1.40 mm to (15.1, 18.4)
- moved R7 1.40 mm to (14.9, 15.2)
- moved 12V-5V-BUCK 0.97 mm to (31.2, 3.05)
- moved F2 0.89 mm to (18.9, 4.19)
- moved FLOW 0.89 mm to (9.02, 3.94)
- moved V2 0.89 mm to (16.5, 3.17)
Connections:
- removed net N$1: JP1.1, R7.1, WATCHDOG.1
- net DELAY: now also R1.2
- net GND: now also R1.1
- net VCC: now also R7.1, WATCHDOG.1; no longer JP1.2
Routing:
- net VCC: track 28.5 -> 39.0 mm
- net N$1: track 8.30 -> 0.00 mm
- net DELAY: track 2.84 -> 6.22 mm
- net LOAD-GND: track 30.7 -> 32.3 mm
- net !RST: track 26.4 -> 27.7 mm
- net WAKE: track 22.0 -> 23.1 mm
- net DONE: track 10.0 -> 9.03 mm
- net VIN: track 23.9 -> 24.6 mm
Other:
- board text added: "DC-IN GND"
- board text added: "chip@seeinsights.com 9-12-17 AquaMaster Carrier v2"
- board text removed: "chip@seeinsights.com 8-22-17 AquaMaster Carrier v2"
