File: AquaMaster-Carrier.sch (EAGLE design)
At the start: 44 parts, among them J2 5V @ 2A, Q1 BSS138, Q2 BSS138, Q3 BSS138, Q4 BSS138

Commit message: Latest AquaMaster Carrier Board - sent to OSHPark today
Parts:
- removed JP2: VSelect, SparkFun-Jumpers:JUMPER-SMT_3_1-NC_PASTE_SILK
- removed Q1, Q2, Q3, Q4: BSS138, SparkFun:MOSFET-NCHANNELSMD
- removed R1, R10, R11, R12, R4, R6, R8, R9: 10K, adafruit:R-US_R0805
- removed SPI: (no value), SparkFun-Connectors:CONN_06LOCK
- added FLOW: (no value), SparkFun-Connectors:CONN_03LOCK
Connections:
- removed net A2-EXT: Q1.D, R4.2, SPI.2
- removed net A3: PHOTON.A3, Q2.S, R6.2
- removed net A3-EXT: Q2.D, R8.2, SPI.3
- removed net A4: PHOTON.A4, Q3.S, R9.2
- removed net A4-EXT: Q3.D, R10.2, SPI.4
- removed net A5: PHOTON.A5, Q4.S, R11.2
- removed net A5-EXT: Q4.D, R12.2, SPI.5
- removed net VIO-EXT: F2.2, SPI.6, V2.2
- removed net VSELECT: F2.1, JP2.2, R10.1, R12.1, R4.1, R8.1
- new net LED: PHOTON.D7
- new net VIN-EXT: F2.2, FLOW.3, V2.2
- net A2: now also FLOW.2; no longer Q1.S, R1.2
- net DONE: now also PHOTON.D2; no longer PHOTON.D6
- net GND: now also FLOW.1; no longer SPI.1
- net SOLENOID: now also PHOTON.D6; no longer PHOTON.D2
- net VCC: no longer JP2.3, Q1.G, Q2.G, Q3.G, Q4.G, R1.1, R11.1, R13.2, R14.2, R6.1, R9.1
- net VCC-EXT: now also R13.2, R14.2
- net VIN: now also F2.1; no longer JP2.1
Other:
- note added: "AquaMaster Carrier Board"
- note added: "DC-IN - 12V @3.5A Vin - 5V @ 1.5A Vcc - 3.3V @100mA Murata Buck Converter used: http://power.murata.com/data/power/oki-78sr.pdf"
- note removed: "DC-IN - 12V @3.5A Vin - 5V @ 1.5A Vcc - 3.3V @100mA VIO is either 3.3V or 5V based on VSelect Murata Buck Converter used: http://power.murata.com/data/power/oki-78sr.pdf"
- note removed: "IO Pins either 3.3V (Vcc) or 5V (Vin) with this VSelect solder jumper"
- note removed: "Note: A5 cannor be an external interrupt pin"
- note removed: "Note: If ESD / Overvoltage protection is not needed, leave Varisors unpopulated and replace fuses with 1206 zero ohm resistors or jumper wire."
- note removed: "SPI Bus Level Shifters"
- moved on the sheet: 12V-5V-BUCK, C1, D-IO, F1, F2, F3, I2C, J2, R13, R14, V1, V2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

Commit message: Added BOM
Parts:
- removed JP1: DOG-SW, SparkFun-Jumpers:JUMPER-SMT_2_NO_NO-SILK
- added LOGO1: OSHW-LOGOS, SparkFun-Aesthetics:OSHW-LOGOS
- added R1: 97.6k, adafruit:R-US_R0805
- R2: value 25k -> 100k
Connections:
- removed net N$1: JP1.1, R7.1, WATCHDOG.VDD
- net DELAY: now also R1.2
- net GND: now also R1.1
- net VCC: now also R7.1, WATCHDOG.VDD; no longer JP1.2
Other:
- note added: "Note: R1 and R2 values set the interval of the watchdog interrupts. See datasheet. Values provided here yeild a 7min interval."
- note added: "v2.1"
- note removed: "Note: Watchdog is optional or you can install and solder the jumper when ready."
- note removed: "v2"
- moved on the sheet: R2, R7, WATCHDOG
Changed lines of the file:
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@@
 <?xml version="1.0" encoding="utf-8"?>
 <!DOCTYPE eagle SYSTEM "eagle.dtd">
-<eagle version="8.3.0">
+<eagle version="8.3.2">
 <drawing>
 <settings>
@@
 <part name="R3" library="adafruit" deviceset="R-US_" device="R0805" value="1k"/>
 <part name="C1" library="SparkFun-Capacitors" deviceset="1.0UF" device="-0805-25V-10%" value="1.0uF"/>
-<part name="R2" library="adafruit" deviceset="R-US_" device="R0805" value="25k"/>
+<part name="R2" library="adafruit" deviceset="R-US_" device="R0805" value="100k"/>
 <part name="GND1" library="SparkFun-PowerSymbols" deviceset="GND" device=""/>
 <part name="R7" library="adafruit" deviceset="R-US_" device="R0805" value="100k"/>
@@
 <part name="F2" library="SparkFun-Fuses" deviceset="PPTC" device="_HALF-AMP" value="500mA - FAST BLOW"/>
 <part name="D-IO" library="SparkFun-Connectors" deviceset="CONN_04" device="LOCK"/>
-<part name="JP1" library="SparkFun-Jumpers" deviceset="JUMPER-SMT_2_NO" device="_NO-SILK" value="DOG-SW"/>
 <part name="SUPPLY2" library="SparkFun-PowerSymbols" deviceset="VCC" device=""/>
 <part name="FLOW" library="SparkFun-Connectors" deviceset="CONN_03" device="LOCK"/>
+<part name="R1" library="adafruit" deviceset="R-US_" device="R0805" value="97.6k"/>
+<part name="LOGO1" library="SparkFun-Aesthetics" deviceset="OSHW-LOGO" device="S"/>
 </parts>
 <sheets>
@@
 <plain>
 <text x="172.72" y="7.62" size="3.81" layer="94">Chip McClelland</text>
-<text x="241.3" y="7.62" size="3.81" layer="94">v2</text>
+<text x="236.22" y="7.62" size="3.81" layer="94">v2.1</text>
 <text x="160.02" y="38.1" size="1.778" layer="91">DC-IN - 12V @3.5A
 Vin - 5V @ 1.5A
@@
 <text x="53.34" y="170.18" size="1.778" layer="97" rot="R180">On-Board Components</text>
 <text x="231.14" y="170.18" size="1.778" layer="97" rot="R180">Particle Photon and External Connections</text>
-<text x="2.54" y="60.96" size="1.778" layer="91">Note: Watchdog is optional or you can install
-and solder the jumper when ready.</text>
+<text x="2.54" y="60.96" size="1.778" layer="91">Note: R1 and R2 values set the
+interval of the watchdog interrupts.  See datasheet.
+Values provided here yeild a 7min interval.</text>
 <text x="167.64" y="180.34" size="5.08" layer="97" rot="R180">AquaMaster Carrier Board</text>
 </plain>
@@
 <instance part="R14" gate="G$1" x="241.3" y="96.52" rot="R90"/>
 <instance part="SWITCH" gate="G$1" x="45.72" y="137.16"/>
-<instance part="WATCHDOG" gate="G$1" x="43.18" y="83.82"/>
+<instance part="WATCHDOG" gate="G$1" x="43.18" y="91.44"/>
 <instance part="R5" gate="G$1" x="33.02" y="127" rot="R90"/>
 <instance part="GND2" gate="1" x="27.94" y="119.38"/>
@@
 <instance part="R3" gate="G$1" x="20.32" y="132.08"/>
 <instance part="C1" gate="G$1" x="228.6" y="134.62"/>
-<instance part="R2" gate="G$1" x="15.24" y="78.74"/>
+<instance part="R2" gate="G$1" x="15.24" y="86.36"/>
 <instance part="GND1" gate="1" x="10.16" y="71.12"/>
-<instance part="R7" gate="G$1" x="53.34" y="101.6"/>
+<instance part="R7" gate="G$1" x="53.34" y="109.22"/>
 <instance part="J1" gate="G$1" x="30.48" y="154.94"/>
 <instance part="I2C" gate="G$1" x="73.66" y="17.78"/>
@@
 <instance part="J2" gate="G$1" x="93.98" y="83.82" rot="R90"/>
 <instance part="F3" gate="G$1" x="114.3" y="86.36"/>
-<instance part="JP1" gate="G$1" x="20.32" y="106.68" rot="R90"/>
 <instance part="SUPPLY2" gate="G$1" x="20.32" y="114.3"/>
 <instance part="FLOW" gate="J$1" x="33.02" y="20.32"/>
+<instance part="R1" gate="G$1" x="15.24" y="78.74"/>
+<instance part="LOGO1" gate="G$1" x="121.92" y="43.18"/>
 </instances>
 <busses>
@@
 <segment>
 <pinref part="R2" gate="G$1" pin="1"/>
-<wire x1="10.16" y1="78.74" x2="10.16" y2="73.66" width="0.1524" layer="91"/>
+<wire x1="10.16" y1="86.36" x2="10.16" y2="78.74" width="0.1524" layer="91"/>
 <pinref part="GND1" gate="1" pin="GND"/>
 <pinref part="WATCHDOG" gate="G$1" pin="GND"/>
-<label x="22.86" y="83.82" size="1.778" layer="95"/>
-<wire x1="30.48" y1="83.82" x2="10.16" y2="83.82" width="0.1524" layer="91"/>
-<wire x1="10.16" y1="83.82" x2="10.16" y2="78.74" width="0.1524" layer="91"/>
+<label x="22.86" y="91.44" size="1.778" layer="95"/>
+<wire x1="30.48" y1="91.44" x2="10.16" y2="91.44" width="0.1524" layer="91"/>
+<wire x1="10.16" y1="91.44" x2="10.16" y2="86.36" width="0.1524" layer="91"/>
+<junction x="10.16" y="86.36"/>
+<pinref part="R1" gate="G$1" pin="1"/>
 <junction x="10.16" y="78.74"/>
+<wire x1="10.16" y1="78.74" x2="10.16" y2="73.66" width="0.1524" layer="91"/>
 </segment>
 <segment>
@@
 </segment>
 <segment>
-<pinref part="JP1" gate="G$1" pin="2"/>
 <pinref part="SUPPLY2" gate="G$1" pin="VCC"/>
-<wire x1="20.32" y1="111.76" x2="20.32" y2="114.3" width="0.1524" layer="91"/>
+<wire x1="20.32" y1="109.22" x2="20.32" y2="114.3" width="0.1524" layer="91"/>
+<pinref part="WATCHDOG" gate="G$1" pin="VDD"/>
+<wire x1="30.48" y1="96.52" x2="20.32" y2="96.52" width="0.1524" layer="91"/>
+<wire x1="20.32" y1="96.52" x2="20.32" y2="109.22" width="0.1524" layer="91"/>
+<wire x1="20.32" y1="109.22" x2="48.26" y2="109.22" width="0.1524" layer="91"/>
+<pinref part="R7" gate="G$1" pin="1"/>
+<junction x="20.32" y="109.22"/>
 </segment>
 </net>
@@
 <segment>
 <pinref part="WATCHDOG" gate="G$1" pin="RST"/>
-<wire x1="58.42" y1="88.9" x2="66.04" y2="88.9" width="0.1524" layer="91"/>
-<label x="60.96" y="88.9" size="1.778" layer="95"/>
+<wire x1="58.42" y1="96.52" x2="66.04" y2="96.52" width="0.1524" layer="91"/>
+<label x="60.96" y="96.52" size="1.778" layer="95"/>
 <pinref part="R7" gate="G$1" pin="2"/>
-<wire x1="58.42" y1="101.6" x2="58.42" y2="88.9" width="0.1524" layer="91"/>
-<junction x="58.42" y="88.9"/>
+<wire x1="58.42" y1="109.22" x2="58.42" y2="96.52" width="0.1524" layer="91"/>
+<junction x="58.42" y="96.52"/>
 </segment>
 <segment>
@@
 <segment>
 <pinref part="WATCHDOG" gate="G$1" pin="DELAY"/>
-<label x="22.86" y="78.74" size="1.778" layer="95"/>
+<label x="22.86" y="86.36" size="1.778" layer="95"/>
 <pinref part="R2" gate="G$1" pin="2"/>
-<wire x1="20.32" y1="78.74" x2="30.48" y2="78.74" width="0.1524" layer="91"/>
+<wire x1="20.32" y1="86.36" x2="30.48" y2="86.36" width="0.1524" layer="91"/>
+<pinref part="R1" gate="G$1" pin="2"/>
+<wire x1="20.32" y1="78.74" x2="20.32" y2="86.36" width="0.1524" layer="91"/>
+<junction x="20.32" y="86.36"/>
 </segment>
 </net>
@@
 <segment>
 <pinref part="WATCHDOG" gate="G$1" pin="WAKE"/>
-<wire x1="58.42" y1="83.82" x2="66.04" y2="83.82" width="0.1524" layer="91"/>
-<label x="60.96" y="83.82" size="1.778" layer="95"/>
+<wire x1="58.42" y1="91.44" x2="66.04" y2="91.44" width="0.1524" layer="91"/>
+<label x="60.96" y="91.44" size="1.778" layer="95"/>
 </segment>
 </net>
@@
 <segment>
 <pinref part="WATCHDOG" gate="G$1" pin="DONE"/>
-<wire x1="58.42" y1="78.74" x2="66.04" y2="78.74" width="0.1524" layer="91"/>
-<label x="60.96" y="78.74" size="1.778" layer="95"/>
+<wire x1="58.42" y1="86.36" x2="66.04" y2="86.36" width="0.1524" layer="91"/>
+<label x="60.96" y="86.36" size="1.778" layer="95"/>
 </segment>
 <segment>
@@
 </segment>
 </net>
-<net name="N$1" class="0">
-<segment>
-<pinref part="WATCHDOG" gate="G$1" pin="VDD"/>
-<wire x1="30.48" y1="88.9" x2="20.32" y2="88.9" width="0.1524" layer="91"/>
-<wire x1="20.32" y1="88.9" x2="20.32" y2="101.6" width="0.1524" layer="91"/>
-<wire x1="20.32" y1="101.6" x2="48.26" y2="101.6" width="0.1524" layer="91"/>
-<pinref part="R7" gate="G$1" pin="1"/>
-<pinref part="JP1" gate="G$1" pin="1"/>
-<junction x="20.32" y="101.6"/>
-</segment>
-</net>
