File: Particle-Photon-Carrier.sch (EAGLE design)
At the start: 44 parts, among them J2 5V @ 2A, Q1 BSS138, Q2 BSS138, Q3 BSS138, Q4 BSS138

Commit message: v3 of the AquaMaster
For Spring 2018
Parts:
- removed 12V-5V-BUCK: I50115, SparkFun-Connectors:CONN_03LOCK
- removed D-IO, I2C: (no value), SparkFun-Connectors:CONN_04LOCK
- removed JP1: DOG-SW, SparkFun-Jumpers:JUMPER-SMT_2_NO_NO-SILK
- removed JP2: VSelect, SparkFun-Jumpers:JUMPER-SMT_3_1-NC_PASTE_SILK
- removed Q1, Q2, Q3, Q4: BSS138, SparkFun:MOSFET-NCHANNELSMD
- removed SPI: (no value), SparkFun-Connectors:CONN_06LOCK
- added ANALOG, DIGITAL: (no value), SparkFun-Connectors:CONN_083.5MM-8
- added D2: 3A/40V/500mV, SparkFun-DiscreteSemi:DIODE-SCHOTTKY-B340A
- added F4: 500mA - FAST BLOW, SparkFun-Fuses:PPTC_HALF-AMP
- added J3: (no value), SparkFun-Connectors:CONN_03LOCK
- added J4: (no value), SparkFun-Connectors:CONN_023.5MM
- added LED1, LED2: (no value), adafruit:LEDCHIPLED_0805
- added R15, R16, R17, R18, R19: 1k, adafruit:R-US_R0805
- added SWITCH1: IRF6201PBF, MOSFETs:IRF6201PBF
- added TVS-DIODE: D5V0L4B5TS, Custom Components:D5V0L4B5TS
- added V4: VC080505C150DP, Custom Components:VARISTOR
- J1: device SparkFun-Connectors:CONN_02 -> SparkFun-Connectors:CONN_023.5MM
- R1: value 10K -> 100k
- R10, R11, R12, R4, R6, R8, R9: value 10K -> 1k
Connections:
- net SOLENOID renamed SOLENOID1
- removed net A2-EXT: Q1.D, R4.2, SPI.2
- removed net A3-EXT: Q2.D, R8.2, SPI.3
- removed net A4-EXT: Q3.D, R10.2, SPI.4
- removed net A5-EXT: Q4.D, R12.2, SPI.5
- removed net VCC-EXT: D-IO.4, F1.2, I2C.4, V1.2
- removed net VIO-EXT: F2.2, SPI.6, V2.2
- removed net VSELECT: F2.1, JP2.2, R10.1, R12.1, R4.1, R8.1
- new net A0: PHOTON.A0
- new net A1: PHOTON.A1, R15.1
- new net D5: PHOTON.D5, R18.1
- new net DAC: PHOTON.DAC, R8.1
- new net EXT-A1: ANALOG.7, R15.2
- new net EXT-A2: ANALOG.6, R12.2
- new net EXT-A3: ANALOG.5, R11.2
- new net EXT-A4: ANALOG.4, R10.2
- new net EXT-A5: ANALOG.3, R9.2
- new net EXT-D3: DIGITAL.5, R16.2
- new net EXT-D4: DIGITAL.6, R17.2
- new net EXT-D5: DIGITAL.7, R18.2
- new net EXT-DAC: ANALOG.2, R8.2
- new net GATE1: R1.2, R4.2, SWITCH1.G
- new net LOAD-GND2: D2.A, J4.1, R6.2, SWITCH1.D1, SWITCH1.D2, SWITCH1.D3, SWITCH1.D4
- new net N$2: LED1.C, R19.2
- new net RX: PHOTON.RX
- new net SOLENOID2: PHOTON.D7, R4.1
- new net TX: PHOTON.TX
- new net VCC1-EXT: ANALOG.1, F1.2, LED1.A, V1.2
- new net VCC2-EXT: DIGITAL.1, F2.2, R13.2, R14.2, V2.2
- new net VIN-EXT: DIGITAL.8, F4.2, V4.2
- net A2: now also R12.1; no longer Q1.S, R1.2
- net A3: now also R11.1; no longer Q2.S, R6.2
- net A4: now also R10.1; no longer Q3.S, R9.2
- net A5: now also R9.1; no longer Q4.S, R11.2
- net D3: now also R16.1, TVS-DIODE.5; no longer D-IO.2
- net D4: now also R17.1, TVS-DIODE.4; no longer D-IO.3
- net DC-IN: now also D2.C, J1.1, J3.3, J4.2; no longer 12V-5V-BUCK.3, J1.2
- net GND: now also ANALOG.8, DIGITAL.4, J3.2, PHOTON.GND@2, R1.1, SWITCH1.S1, SWITCH1.S2, SWITCH1.S3, TVS-DIODE.GND, V4.1; no longer 12V-5V-BUCK.2, D-IO.1, I2C.1, SPI.1
- net LOAD-GND: now also J1.2, R19.1; no longer J1.1
- net N$1: now also LED2.C, R6.1; no longer JP1.1, R7.1, WATCHDOG.VDD
- net SCL: now also DIGITAL.3, TVS-DIODE.1; no longer I2C.3
- net SDA: now also DIGITAL.2, TVS-DIODE.3; no longer I2C.2
- net VCC: now also F2.1, LED2.A, R7.1, WATCHDOG.VDD; no longer JP1.2, JP2.3, Q1.G, Q2.G, Q3.G, Q4.G, R1.1, R11.1, R13.2, R14.2, R6.1, R9.1
- net VIN: now also F4.1, J3.1; no longer 12V-5V-BUCK.1, JP2.1
Other:
- note added: "All 1k ohm"
- note added: "DC-IN - 12V @3.5A Vin - 5V @ 1.5A Vcc - 3.3V @800mA"
- note added: "Note: A5 cannot be an external interrupt pin"
- note added: "v3"
- note removed: "DC-IN - 12V @3.5A Vin - 5V @ 1.5A Vcc - 3.3V @100mA VIO is either 3.3V or 5V based on VSelect Murata Buck Converter used: http://power.murata.com/data/power/oki-78sr.pdf"
- note removed: "IO Pins either 3.3V (Vcc) or 5V (Vin) with this VSelect solder jumper"
- note removed: "Note: A5 cannor be an external interrupt pin"
- note removed: "Note: Watchdog is optional or you can install and solder the jumper when ready."
- note removed: "SPI Bus Level Shifters"
- note removed: "v2"
- moved on the sheet: C1, D1, F1, F2, J1, R1, R10, R11, R12, R2, R3, R4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
